Commit message: A lot of changes

File: panda_description/urdf/include/mir.gazebo.xacro (robot description, xacro)
@@ -1,5 +1,5 @@
 <?xml version="1.0"?>
 <robot xmlns:xacro="http://www.ros.org/wiki/xacro">
-    <ros2_control name="GazeboSimSystem" type="system">
+    <!-- <ros2_control name="GazeboSimSystem" type="system">
         <hardware>
             <plugin>gz_ros2_control/GazeboSimSystem</plugin>
@@ -15,5 +15,5 @@
             <state_interface name="velocity"/>
         </joint>
-    </ros2_control>
+    </ros2_control> -->
     <xacro:macro name="set_wheel_friction" params="link friction">
         <gazebo reference="${link}">

File: panda_description/urdf/mir.urdf.xacro (robot description, xacro)
@@ -30,11 +30,5 @@
     <xacro:property name="laser_dx" value="0.392" />
     <xacro:property name="laser_dy" value="0.2358" />
-    <link name="base_footprint" />
-    <joint name="base_joint" type="fixed">
-      <parent link="base_footprint" />
-      <child link="base_link" />
-      <origin xyz="0 0 0" rpy="0 0 0" />
-    </joint>
-    <link name="base_link">
+    <link name="mir_base">
       <xacro:box_inertial mass="${mir_base_mass}" x="${mir_base_inertial_x_length}" y="${mir_base_inertial_y_length}" z="${mir_base_inertial_z_length}">
         <origin xyz="${mir_base_inertial_x + mir_act_wheel_dx} ${mir_base_inertial_y} ${mir_base_inertial_z}" rpy="0 0 0" />
@@ -54,5 +48,5 @@
       </collision>
     </link>
-    <gazebo reference="base_link">
+    <gazebo reference="mir_base">
       <material>Gazebo/White</material>
     </gazebo>
@@ -60,5 +54,5 @@
       <joint name="${locationprefix}_wheel_joint" type="continuous">
           <origin xyz="0.0 ${-mir_act_wheel_dy * locationright} ${mir_act_wheel_radius}" rpy="0 0 0" />
-          <parent link="base_link" />
+          <parent link="mir_base" />
           <child link="${locationprefix}_wheel_link" />
           <axis xyz="0 1 0" />
@@ -91,5 +85,5 @@
       <joint name="${locationprefix}_caster_rotation_joint" type="continuous">
           <origin xyz="${wheel_base_dx} ${-mir_caster_wheel_base_dy * locationright} ${mir_caster_wheel_base_dz}" rpy="0 0 0" />
-          <parent link="base_link" />
+          <parent link="mir_base" />
           <child link="${locationprefix}_caster_rotation_link" />
           <axis xyz="0 0 1" />

File: panda_description/urdf/panda.urdf (robot description, URDF)
Before this commit: robot panda, 26 links, 25 joints
Links:
- removed link base_link
- removed link panda_mount_plate
- added link box, mass 1.0; collision box size=0.5 0.5 0.3; visual box size=0.5 0.5 0.4
- added link mir_base, mass 77.0; collision mesh filename=file:///home/aayush/Internship/franka1_ws/install/share/pan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; visual mesh filename=file:///home/aayush/Internship/franka1_ws/install/share/pan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
- link bl_caster_rotation_link: geometry collision mesh filename=file:///home/aayush/Internship/franka1_ws/install/share/pan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; visual mesh filename=file:///home/aayush/Internship/franka1_ws/install/share/pan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
- link br_caster_rotation_link: geometry collision mesh filename=file:///home/aayush/Internship/franka1_ws/install/share/pan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; visual mesh filename=file:///home/aayush/Internship/franka1_ws/install/share/pan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
- link fl_caster_rotation_link: geometry collision mesh filename=file:///home/aayush/Internship/franka1_ws/install/share/pan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; visual mesh filename=file:///home/aayush/Internship/franka1_ws/install/share/pan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
- link fr_caster_rotation_link: geometry collision mesh filename=file:///home/aayush/Internship/franka1_ws/install/share/pan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; visual mesh filename=file:///home/aayush/Internship/franka1_ws/install/share/pan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
Joints:
- removed joint mir_to_mount_plate_joint
- removed joint world_to_mir_joint
- added joint base_joint_box: type fixed, parent world, child mir_base, origin xyz=0 0 -0.65 rpy=0 0 0
- added joint some_joint: type fixed, parent world, child box, origin xyz=0.0 0.0 -0.2 rpy=0.0 0.0 0.0
- joint bl_caster_rotation_joint: parent base_link -> mir_base
- joint br_caster_rotation_joint: parent base_link -> mir_base
- joint fl_caster_rotation_joint: parent base_link -> mir_base
- joint fr_caster_rotation_joint: parent base_link -> mir_base
- joint left_wheel_joint: parent base_link -> mir_base
- joint panda_joint_base: origin xyz=0 0 0.05 rpy=0 0 0 -> xyz=0 0 0 rpy=0 0 0; parent panda_mount_plate -> world
- joint right_wheel_joint: parent base_link -> mir_base

File: panda_description/urdf/panda.urdf.xacro (robot description, xacro)
@@ -9,4 +9,5 @@
   <xacro:include filename="$(find panda_description)/urdf/panda_utils.xacro"/>
   <xacro:include filename="$(find panda_description)/urdf/panda.gazebo"/>
+  <xacro:include filename="$(find panda_description)/urdf/mir.urdf.xacro"/>
   <!--            -->
   <!-- Parameters -->
@@ -63,7 +64,7 @@
   <!-- Arm -->
   <xacro:panda_arm
-    base_parent="panda_mount_plate"
+    base_parent="${world_name}"
     prefix="${prefix_arm}"
-    origin_xyz="0 0 0.05"
+    origin_xyz="${origin_xyz}"
     origin_rpy="${origin_rpy}"
     collision="$(arg collision_arm)"
@@ -97,32 +98,20 @@
     </xacro:if>
   </xacro:if>
-  <!-- Mounting parameters for Panda on MiR -->
-  <xacro:arg name="panda_mount_height" default="0.35"/>  <!-- Height above MiR base -->
-  <xacro:arg name="panda_mount_x" default="0.0"/>       <!-- X offset from MiR center -->
-  <xacro:arg name="panda_mount_y" default="0.0"/>       <!-- Y offset from MiR center -->
-  <xacro:include filename="$(find panda_description)/urdf/mir.urdf.xacro"/>
-  <!-- <link name="${world_name}"/> -->
-  <!-- MiR mobile base -->
   <xacro:mir/>
-  <!-- Fixed joint connecting world to MiR base -->
-  <joint name="world_to_mir_joint" type="fixed">
-    <parent link="${world_name}"/>
-    <child link="base_footprint"/>
-    <origin xyz="0 0 0.05" rpy="${origin_rpy}"/>
-  </joint>
-  <!-- Mounting plate link -->
-  <link name="panda_mount_plate">
+  <link name="box">
     <inertial>
       <origin xyz="0 0 0" rpy="0 0 0"/>
-      <mass value="5.0"/>
-      <inertia ixx="0.1" ixy="0" ixz="0" iyy="0.1" iyz="0" izz="0.1"/>
+      <mass value="1.0"/> <!-- non-zero mass -->
+      <inertia ixx="0.01" ixy="0.0" ixz="0.0"
+              iyy="0.01" iyz="0.0"
+              izz="0.01"/>
     </inertial>
-    <visual>
+    <visual name="box_visual">
       <origin xyz="0 0 0" rpy="0 0 0"/>
       <geometry>
-        <box size="0.3 0.3 0.05"/>
+        <box size="0.5 0.5 0.4"/>
       </geometry>
-      <material name="mount_plate_color">
-        <color rgba="0.8 0.8 0.8 1.0"/>
+      <material name="Grey">
+        <color rgba="0.5 0.5 0.5 1.0"/>
       </material>
     </visual>
@@ -130,13 +119,20 @@
       <origin xyz="0 0 0" rpy="0 0 0"/>
       <geometry>
-        <box size="0.3 0.3 0.05"/>
+        <box size="0.5 0.5 0.3"/>
       </geometry>
     </collision>
   </link>
-  <!-- Fixed joint mounting the plate to MiR base -->
-  <joint name="mir_to_mount_plate_joint" type="fixed">
-    <parent link="base_link"/>
-    <child link="panda_mount_plate"/>
-    <origin xyz="$(arg panda_mount_x) $(arg panda_mount_y) $(arg panda_mount_height)" rpy="0 0 0"/>
+  <gazebo reference="box">
+    <material>Gazebo/Grey</material>
+  </gazebo>
+  <joint name="base_joint_box" type="fixed">
+    <origin xyz="-0.1 0 -0.65" rpy="0 0 0"/>
+    <parent link="${world_name}"/>
+    <child link="mir_base"/>
+  </joint>
+  <joint name="some_joint" type="fixed">
+    <origin xyz="-0.1 0.0 -0.2" rpy="0.0 0.0 0.0"/>
+    <parent link="${world_name}"/>
+    <child link="box"/>
   </joint>
 </robot>

File: panda_description/urdf/panda_gripper.xacro (robot description, xacro)
@@ -133,4 +133,67 @@
     gazebo_preserve_fixed_joint="${gazebo_preserve_fixed_joint}"
     />
+    <!-- Main brush body -->
+    <link name="mirror_brush_body">
+      <inertial>
+        <origin xyz="0 0 0.05" rpy="0 0 0"/>
+        <mass value="0.15"/>
+        <inertia ixx="0.0008" ixy="0" ixz="0" iyy="0.0015" iyz="0" izz="0.0008"/>
+      </inertial>
+      <!-- Ergonomic Handle (blue plastic) -->
+      <visual>
+        <origin xyz="0 0 0.075" rpy="0 0 0"/>
+        <geometry>
+          <cylinder radius="0.015" length="0.07"/>
+        </geometry>
+        <material name="blue_handle">
+          <color rgba="0.1 0.3 0.7 1"/>
+        </material>
+      </visual>
+      <collision>
+        <origin xyz="0 0 0.075" rpy="0 0 0"/>
+        <geometry>
+          <cylinder radius="0.015" length="0.07"/>
+        </geometry>
+      </collision>
+      <!-- Handle grip -->
+      <visual>
+        <origin xyz="0 0 0.05" rpy="0 0 0"/>
+        <geometry>
+          <cylinder radius="0.017" length="0.03"/>
+        </geometry>
+        <material name="dark_rubber">
+          <color rgba="0.2 0.2 0.2 1"/>
+        </material>
+      </visual>
+      <!-- Brush head (rotated & enlarged) -->
+      <visual>
+        <origin xyz="0 0 0.0" rpy="1.5708 0 0"/>
+        <geometry>
+          <box size="0.09 0.055 0.015"/>
+        </geometry>
+        <material name="white_head">
+          <color rgba="0.95 0.95 0.95 1"/>
+        </material>
+      </visual>
+      <collision>
+        <origin xyz="0 0 0.0" rpy="1.5708 0 0"/>
+        <geometry>
+          <box size="0.09 0.055 0.015"/>
+        </geometry>
+      </collision>
+      <!-- Simplified collision for bristles -->
+      <collision>
+        <origin xyz="0 0 -0.005" rpy="1.5708 0 0"/>
+        <geometry>
+          <box size="0.08 0.05 0.008"/>
+        </geometry>
+      </collision>
+    </link>
+    <!-- Joint to attach brush to robot end-effector -->
+    <joint name="brush_mount_joint" type="fixed">
+      <parent link="${prefix}${link_finger2_name}"/>
+      <child link="mirror_brush_body"/>
+      <origin xyz="0.0 0.05 0.12" rpy="0 3.1415 0"/>
+    </joint>
     <!-- ROS 2 control -->
     <xacro:if value="${ros2_control}">

File: panda_moveit_config/srdf/panda.srdf.xacro (robot description, xacro)
@@ -30,12 +30,4 @@
   />
   <end_effector group="gripper" name="gripper" parent_group="arm" parent_link="${prefix_arm}hand_tcp"/>
-  <passive_joint name="bl_caster_rotation_joint"/>
-  <passive_joint name="bl_caster_wheel_joint"/>
-  <passive_joint name="br_caster_rotation_joint"/>
-  <passive_joint name="br_caster_wheel_joint"/>
-  <passive_joint name="fl_caster_rotation_joint"/>
-  <passive_joint name="fl_caster_wheel_joint"/>
-  <passive_joint name="fr_caster_rotation_joint"/>
-  <passive_joint name="fr_caster_wheel_joint"/>
   <disable_collisions link1="${prefix_gripper}hand" link2="${prefix_arm}link3" reason="Never"/>
   <disable_collisions link1="${prefix_gripper}hand" link2="${prefix_arm}link4" reason="Never"/>
